File: sensor.kicad_sch (KiCad schematic)
At the start: 8 parts, among them U2 ICM-42688-P

Commit message: routing...
Parts:
- U3: footprint fcg4_fp:SENSOR-SMD_SPL06-001 -> ProLib_pcs_2026-02-12:SENSOR-SMD_SPL06-001
Changed lines of the file:
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@@
 			)
 		)
-		(property "Footprint" "fcg4_fp:SENSOR-SMD_SPL06-001"
+		(property "Footprint" "ProLib_pcs_2026-02-12:SENSOR-SMD_SPL06-001"
 			(at 222.25 42.164 0)
 			(effects

Commit message: Update footprint references and component values in schematic files
- Changed footprint property for a component in mcu.kicad_sch from "Package_DFN_QFN:QFN-48-1EP_7x7mm_P0.5mm_EP5.6x5.6mm" to "fcg4_fp:QFN-48-1EP_7x7mm_P0.5mm_EP5.6x5.6mm".
- Updated value property for a component in mcu.kicad_sch from "SolderJumper_2_Open" to "BOOT".
- Changed value property for another component in mcu.kicad_sch from "SolderJumper_2_Open" to "RESET".
- Modified footprint property for a component in sensor.kicad_sch from "ProLib_pcs_2026-02-12:SENSOR-SMD_SPL06-001" to "fcg4_fp:SENSOR-SMD_SPL06-001".
Parts:
- U3: footprint ProLib_pcs_2026-02-12:SENSOR-SMD_SPL06-001 -> fcg4_fp:SENSOR-SMD_SPL06-001
Changed lines of the file:
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@@
 			)
 		)
-		(property "Footprint" "ProLib_pcs_2026-02-12:SENSOR-SMD_SPL06-001"
+		(property "Footprint" "fcg4_fp:SENSOR-SMD_SPL06-001"
 			(at 222.25 42.164 0)
 			(effects
