File: sensor.kicad_sch (KiCad schematic)
At the start: 8 parts, among them U2 ICM-42688-P

Commit message: Almost completed! Update component properties in sensor schematic
- Added datasheets, LCSC part names, manufacturer names, and manufacturer part numbers for various components in the sensor.kicad_sch file.
- Updated the datasheet links for components to point to the correct URLs.
Parts:
- C26: LCSC Part Name (none) -> C91601; Manufacturer_Name (none) -> muRata; Manufacturer_Part_Number (none) -> GCM155R71H103KA55D
- C28: LCSC Part Name (none) -> C385032; Manufacturer_Name (none) -> muRata; Manufacturer_Part_Number (none) -> GRM155R61E225KE11D
- R14: LCSC Part Name (none) -> C60491; Manufacturer_Name (none) -> YAGEO; Manufacturer_Part_Number (none) -> RC0402FR-07100KL
- U2: LCSC Part Name (none) -> C1850418; Manufacturer_Name (none) -> TDK InvenSense; Manufacturer_Part_Number (none) -> ICM-42688-P
- U3: LCSC Part Name 普通气压传感器 停产 -> C2684428; Manufacturer_Name (none) -> Goertek; Manufacturer_Part_Number (none) -> SPL06-001
Changed lines of the file:
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@@
 			)
 		)
-		(property "Datasheet" ""
+		(property "Datasheet" "https://www.lcsc.com/datasheet/C1850418.pdf"
 			(at 78.74 50.8 0)
 			(effects
@@
 				)
 				(justify bottom)
+				(hide yes)
+			)
+		)
+		(property "LCSC Part Name" "C1850418"
+			(at 78.74 50.8 0)
+			(effects
+				(font
+					(size 1.27 1.27)
+				)
+				(hide yes)
+			)
+		)
+		(property "Manufacturer_Name" "TDK InvenSense"
+			(at 78.74 50.8 0)
+			(effects
+				(font
+					(size 1.27 1.27)
+				)
+				(hide yes)
+			)
+		)
+		(property "Manufacturer_Part_Number" "ICM-42688-P"
+			(at 78.74 50.8 0)
+			(effects
+				(font
+					(size 1.27 1.27)
+				)
 				(hide yes)
 			)
@@
 			)
 		)
-		(property "Datasheet" "~"
+		(property "Datasheet" "https://www.lcsc.com/datasheet/C60491.pdf"
 			(at 234.95 63.5 0)
 			(effects
@@
 		)
 		(property "Description" "Resistor"
+			(at 234.95 63.5 0)
+			(effects
+				(font
+					(size 1.27 1.27)
+				)
+				(hide yes)
+			)
+		)
+		(property "LCSC Part Name" "C60491"
+			(at 234.95 63.5 0)
+			(effects
+				(font
+					(size 1.27 1.27)
+				)
+				(hide yes)
+			)
+		)
+		(property "Manufacturer_Name" "YAGEO"
+			(at 234.95 63.5 0)
+			(effects
+				(font
+					(size 1.27 1.27)
+				)
+				(hide yes)
+			)
+		)
+		(property "Manufacturer_Part_Number" "RC0402FR-07100KL"
 			(at 234.95 63.5 0)
 			(effects
@@
 			)
 		)
-		(property "Datasheet" "~"
+		(property "Datasheet" "https://www.lcsc.com/datasheet/C385032.pdf"
 			(at 104.14 38.1 0)
 			(effects
@@
 		(property "Description" "Unpolarized capacitor"
 			(at 104.14 38.1 0)
+			(effects
+				(font
+					(size 1.27 1.27)
+				)
+				(hide yes)
+			)
+		)
+		(property "LCSC Part Name" "C385032"
+			(at 104.14 38.1 90)
+			(effects
+				(font
+					(size 1.27 1.27)
+				)
+				(hide yes)
+			)
+		)
+		(property "Manufacturer_Name" "muRata"
+			(at 104.14 38.1 90)
+			(effects
+				(font
+					(size 1.27 1.27)
+				)
+				(hide yes)
+			)
+		)
+		(property "Manufacturer_Part_Number" "GRM155R61E225KE11D"
+			(at 104.14 38.1 90)
 			(effects
 				(font
@@
 			)
 		)
-		(property "Datasheet" "~"
+		(property "Datasheet" "https://www.lcsc.com/datasheet/C91601.pdf"
 			(at 118.11 45.72 0)
 			(effects
@@
 		)
 		(property "Description" "Unpolarized capacitor"
+			(at 118.11 45.72 0)
+			(effects
+				(font
+					(size 1.27 1.27)
+				)
+				(hide yes)
+			)
+		)
+		(property "LCSC Part Name" "C91601"
+			(at 118.11 45.72 0)
+			(effects
+				(font
+					(size 1.27 1.27)
+				)
+				(hide yes)
+			)
+		)
+		(property "Manufacturer_Name" "muRata"
+			(at 118.11 45.72 0)
+			(effects
+				(font
+					(size 1.27 1.27)
+				)
+				(hide yes)
+			)
+		)
+		(property "Manufacturer_Part_Number" "GCM155R71H103KA55D"
 			(at 118.11 45.72 0)
 			(effects
@@
 			)
 		)
-		(property "Datasheet" "https://item.szlcsc.com/datasheet/SPL06-001/2782076.html"
+		(property "Datasheet" "https://www.lcsc.com/datasheet/C2684428.pdf"
 			(at 222.25 62.484 0)
 			(effects
@@
 			)
 		)
-		(property "LCSC Part Name" "普通气压传感器 停产"
+		(property "LCSC Part Name" "C2684428"
 			(at 222.25 65.532 0)
 			(effects
 				(font
+					(size 1.27 1.27)
+				)
+				(hide yes)
+			)
+		)
+		(property "Manufacturer_Name" "Goertek"
+			(at 222.25 53.34 0)
+			(effects
+				(font
+					(size 1.27 1.27)
+				)
+				(hide yes)
+			)
+		)
+		(property "Manufacturer_Part_Number" "SPL06-001"
+			(at 222.25 53.34 0)
+			(effects
+				(font

Commit message: reorganized everything and switched to 0603 as a minimum size
Parts:
- C26, C27, C28, C29, C30: footprint Capacitor_SMD:C_0402_1005Metric -> Capacitor_SMD:C_0603_1608Metric
- R14: footprint Resistor_SMD:R_0402_1005Metric -> Resistor_SMD:R_0603_1608Metric
- U3: footprint fcg4_fp:SENSOR-SMD_SPL06-001 -> ProLib_pcs_2026-02-12:SENSOR-SMD_SPL06-001; LCSC Part Name C2684428 -> 普通气压传感器 停产
Changed lines of the file:
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@@
 		)
 		(instances
-			(project ""
+			(project "fcg4"
 				(path "/ebe93c2f-0aae-4f69-99fc-930f63b0ac94/4b9bfb89-4b08-43bb-8e52-e82396130844"
 					(reference "U2")
@@
 			)
 		)
-		(property "Footprint" "Capacitor_SMD:C_0402_1005Metric"
+		(property "Footprint" "Capacitor_SMD:C_0603_1608Metric"
 			(at 107.95 30.7848 0)
 			(effects
@@
 			)
 		)
-		(property "Datasheet" "https://www.lcsc.com/datasheet/C77020.pdf"
+		(property "Datasheet" "~"
 			(at 104.14 31.75 0)
 			(effects
@@
 			)
 		)
-		(property "Footprint" "Resistor_SMD:R_0402_1005Metric"
+		(property "Footprint" "Resistor_SMD:R_0603_1608Metric"
 			(at 233.172 63.5 90)
 			(effects
@@
 			)
 		)
-		(property "Datasheet" "https://www.lcsc.com/datasheet/C60491.pdf"
+		(property "Datasheet" "~"
 			(at 234.95 63.5 0)
 			(effects
@@
 			)
 		)
-		(property "Footprint" "Capacitor_SMD:C_0402_1005Metric"
+		(property "Footprint" "Capacitor_SMD:C_0603_1608Metric"
 			(at 107.95 37.1348 0)
 			(effects
@@
 			)
 		)
-		(property "Datasheet" "https://www.lcsc.com/datasheet/C385032.pdf"
+		(property "Datasheet" "~"
 			(at 104.14 38.1 0)
 			(effects
@@
 			)
 		)
-		(property "Footprint" "Capacitor_SMD:C_0402_1005Metric"
+		(property "Footprint" "Capacitor_SMD:C_0603_1608Metric"
 			(at 250.4948 50.8 0)
 			(effects
@@
 			)
 		)
-		(property "Datasheet" "https://www.lcsc.com/datasheet/C77020.pdf"
+		(property "Datasheet" "~"
 			(at 251.46 54.61 0)
 			(effects
@@
 		)
 		(instances
-			(project ""
+			(project "fcg4"
 				(path "/ebe93c2f-0aae-4f69-99fc-930f63b0ac94/4b9bfb89-4b08-43bb-8e52-e82396130844"
 					(reference "C29")
@@
 			)
 		)
-		(property "Footprint" "Capacitor_SMD:C_0402_1005Metric"
+		(property "Footprint" "Capacitor_SMD:C_0603_1608Metric"
 			(at 119.0752 49.53 0)
 			(effects
@@
 			)
 		)
-		(property "Datasheet" "https://www.lcsc.com/datasheet/C91601.pdf"
+		(property "Datasheet" "~"
 			(at 118.11 45.72 0)
 			(effects
@@
 		)
 		(instances
-			(project ""
+			(project "fcg4"
 				(path "/ebe93c2f-0aae-4f69-99fc-930f63b0ac94/4b9bfb89-4b08-43bb-8e52-e82396130844"
 					(reference "C26")
@@
 			)
 		)
-		(property "Footprint" "fcg4_fp:SENSOR-SMD_SPL06-001"
+		(property "Footprint" "ProLib_pcs_2026-02-12:SENSOR-SMD_SPL06-001"
 			(at 222.25 42.164 0)
 			(effects
@@
 			)
 		)
-		(property "Datasheet" "https://www.lcsc.com/datasheet/C2684428.pdf"
+		(property "Datasheet" "https://item.szlcsc.com/datasheet/SPL06-001/2782076.html"
 			(at 222.25 62.484 0)
 			(effects
@@
 			)
 		)
-		(property "LCSC Part Name" "C2684428"
+		(property "LCSC Part Name" "普通气压传感器 停产"
 			(at 222.25 65.532 0)
 			(effects
@@
 		)
 		(instances
-			(project ""
+			(project "fcg4"
 				(path "/ebe93c2f-0aae-4f69-99fc-930f63b0ac94/4b9bfb89-4b08-43bb-8e52-e82396130844"
 					(reference "U3")
@@
 		)
 		(instances
-			(project ""
+			(project "fcg4"
 				(path "/ebe93c2f-0aae-4f69-99fc-930f63b0ac94/4b9bfb89-4b08-43bb-8e52-e82396130844"
 					(reference "#PWR019")
@@
 			)
 		)
-		(property "Footprint" "Capacitor_SMD:C_0402_1005Metric"
+		(property "Footprint" "Capacitor_SMD:C_0603_1608Metric"
 			(at 244.1448 50.8 0)
 			(effects
@@
 			)
 		)
-		(property "Datasheet" "https://www.lcsc.com/datasheet/C77020.pdf"
+		(property "Datasheet" "~"
 			(at 245.11 54.61 0)
 			(effects
